File: progrmmable-load/progrmmable-load.sch (KiCad schematic (older format))
At the start: 32 parts, among them J1 Screw_Terminal_01x02, J2 Conn_01x02, Q1 IRLZ44N, SW1 Rotary_Encoder, U1 MCP4725A2T-E_CH, U2 AD8608ARZ-REEL

Commit message: Add R18 to fix LCD contrast
Parts:
- added R18: 2k, Resistor_SMD:R_0603_1608Metric, symbol Device:R
- U1: symbol MCP4725A2T-E_CH:MCP4725A2T-E_CH -> progrmmable-load-rescue:MCP4725A2T-E_CH-MCP4725A2T-E_CH
- U2: symbol 2020-03-03_04-00-48:AD8608ARZ-REEL -> progrmmable-load-rescue:AD8608ARZ-REEL-2020-03-03_04-00-48
Connections:
- net +5V: now also R18.1
- net at DS1.5 (Vo), R16.2: now also R18.2
Other:
- moved on the sheet: R16
Changed lines of the file:
@@
 	3250 3550 3300 3550
 $Comp
-L MCP4725A2T-E_CH:MCP4725A2T-E_CH U1
+L progrmmable-load-rescue:MCP4725A2T-E_CH-MCP4725A2T-E_CH U1
 U 1 1 5E5E2A59
 P 5250 1200
@@
 	4700 2600 4750 2600
 $Comp
-L 2020-03-03_04-00-48:AD8608ARZ-REEL U2
+L progrmmable-load-rescue:AD8608ARZ-REEL-2020-03-03_04-00-48 U2
 U 1 1 5E5F0AE0
 P 6050 4350
@@
 L Device:R R16
 U 1 1 5E7451F3
-P 1500 2050
-F 0 "R16" V 1707 2050 50  0000 C CNN
-F 1 "2k" V 1616 2050 50  0000 C CNN
-F 2 "Resistor_SMD:R_0603_1608Metric" V 1430 2050 50  0001 C CNN
-F 3 "~" H 1500 2050 50  0001 C CNN
-	1    1500 2050
+P 1400 2050
+F 0 "R16" V 1607 2050 50  0000 C CNN
+F 1 "2k" V 1516 2050 50  0000 C CNN
+F 2 "Resistor_SMD:R_0603_1608Metric" V 1330 2050 50  0001 C CNN
+F 3 "~" H 1400 2050 50  0001 C CNN
+	1    1400 2050
 	0    -1   -1   0
 $EndComp
@@
 L power:GND #PWR0125
 U 1 1 5E747A98
-P 1350 2050
-F 0 "#PWR0125" H 1350 1800 50  0001 C CNN
-F 1 "GND" H 1355 1877 50  0000 C CNN
-F 2 "" H 1350 2050 50  0001 C CNN
-F 3 "" H 1350 2050 50  0001 C CNN
-	1    1350 2050
+P 1250 2050
+F 0 "#PWR0125" H 1250 1800 50  0001 C CNN
+F 1 "GND" H 1255 1877 50  0000 C CNN
+F 2 "" H 1250 2050 50  0001 C CNN
+F 3 "" H 1250 2050 50  0001 C CNN
+	1    1250 2050
 	-1   0    0    -1
 $EndComp
@@
 Wire Wire Line
 	4050 2650 3700 2650
+$Comp
+L Device:R R18
+U 1 1 5F13DC30
+P 1600 1850
+F 0 "R18" V 1807 1850 50  0000 C CNN
+F 1 "2k" V 1716 1850 50  0000 C CNN
+F 2 "Resistor_SMD:R_0603_1608Metric" V 1530 1850 50  0001 C CNN
+F 3 "~" H 1600 1850 50  0001 C CNN
+	1    1600 1850
+	1    0    0    -1
+$EndComp
+Wire Wire Line
+	1650 2050 1600 2050
+Wire Wire Line
+	1600 2000 1600 2050
+Connection ~ 1600 2050
+Wire Wire Line
+	1600 2050 1550 2050
+$Comp
+L power:+5V #PWR01
+U 1 1 5F14BEF8
+P 1600 1700
+F 0 "#PWR01" H 1600 1550 50  0001 C CNN
+F 1 "+5V" H 1615 1873 50  0000 C CNN
+F 2 "" H 1600 1700 50  0001 C CNN
+F 3 "" H 1600 1700 50  0001 C CNN
+	1    1600 1700
+	-1   0    0    -1
+$EndComp
 $EndSCHEMATC
